Commit message: Add ROS 2 control and Gazebo launch for wheelchair
- Add wheelchair.yaml ROS 2 control config
- Add wheelchair_gazebo.launch.py and wheelchair.launch.py
- Update robot.urdf with ros2_control and Gazebo plugins
- Define wheel and position controllers for joints

File: wheelchair_ros/wheelchair/robot.urdf (robot description, URDF)
Before this commit: robot nishcorp_wheelchair, 10 links, 9 joints
Links:
- added link world
- link component1: mass 1e-09 -> 3.0
- link component1_2: mass 1e-09 -> 3.0
- link component24_1: mass 1e-09 -> 2.0
- link component24_1_2: mass 1e-09 -> 2.0
- link fiberglass_seat_v3_v9: mass 1e-09 -> 5.0
- link shaft_v2: mass 1e-09 -> 1.0
- link untitled_v1: mass 1e-09 -> 1.0
- link untitled_v1_2: mass 1e-09 -> 1.0
- link zzzzzzz_v1: mass 1e-09 -> 0.5
- link zzzzzzz_v1_2: mass 1e-09 -> 0.5
Joints:
- added joint world_to_base: type fixed, parent world, child fiberglass_seat_v3_v9, origin xyz=0 0 0.5 rpy=0 0 0
- joint j6: limit lower=-3.141592653589793 upper=3.141592653589793 effort=10 velocity=10 -> (none); type revolute -> continuous
- joint j7: limit lower=-3.141592653589793 upper=3.141592653589793 effort=10 velocity=10 -> (none); type revolute -> continuous
- joint j8: limit lower=-3.141592653589793 upper=3.141592653589793 effort=10 velocity=10 -> (none); type revolute -> continuous
- joint j9: limit lower=-3.141592653589793 upper=3.141592653589793 effort=10 velocity=10 -> (none); type revolute -> continuous

Commit message: wheelchair spwaned

File: wheelchair_ros/wheelchair/robot.urdf (robot description, URDF)
Before this commit: robot nishcorp_wheelchair, 11 links, 10 joints
Links:
- removed link world
Joints:
- removed joint world_to_base

Commit message: updated urdf , bot is movable in gazebo

File: wheelchair_ros/wheelchair/robot.urdf (robot description, URDF)
Before this commit: robot nishcorp_wheelchair, 10 links, 9 joints
Links:
- added link base_link, mass 0.1
Joints:
- added joint base_to_seat: type fixed, parent base_link, child fiberglass_seat_v3_v9, origin xyz=0 0 0.3 rpy=0 0 0

Commit message: bot working , joints working

File: wheelchair_ros/wheelchair/robot.urdf (robot description, URDF)
Before this commit: robot nishcorp_wheelchair, 11 links, 10 joints
Joints:
- joint j1: limit lower=-3.14159 upper=0 effort=10 velocity=10 -> lower=-3.14159 upper=0 effort=100 velocity=10
- joint j2: limit lower=0 upper=1.5708 effort=10 velocity=10 -> lower=0 upper=1.5708 effort=100 velocity=10
- joint j3: limit lower=0 upper=1.5708 effort=10 velocity=10 -> lower=0 upper=1.5708 effort=100 velocity=10
- joint j4: limit lower=-1.5708 upper=0 effort=10 velocity=10 -> lower=-1.5708 upper=0 effort=100 velocity=10
- joint j5: limit lower=0 upper=1.5708 effort=10 velocity=10 -> lower=0 upper=1.5708 effort=100 velocity=10

Commit message: Add smooth joint transitions and update URDF inertials
- Implement smooth interpolation for joint movements in
teleop_controller.py - Add stop command and improve wheel control logic
- Update URDF masses and inertias for more realistic simulation

File: wheelchair_ros/wheelchair/robot.urdf (robot description, URDF)
Before this commit: robot nishcorp_wheelchair, 11 links, 10 joints
Links:
- link base_link: mass 0.1 -> 15.0
- link component1: mass 3.0 -> 5.0
- link component1_2: mass 3.0 -> 5.0
- link component24_1: mass 2.0 -> 4.0
- link fiberglass_seat_v3_v9: mass 5.0 -> 8.0
- link shaft_v2: mass 1.0 -> 2.5
- link untitled_v1: mass 1.0 -> 2.0
- link zzzzzzz_v1: mass 0.5 -> 1.0
- link zzzzzzz_v1_2: mass 0.5 -> 1.0
